File: SensoresUS/SensoresUS.kicad_pcb (KiCad board)
At the start: 2 copper layers, 30 parts

Commit message: Placa SUS
Cambio de integrados
Parts:
- removed the Echo1 at (61.0, 127.0)
- removed the Echo1 at (130.8, 74.9)
- removed the Echo1 at (45.7, 163.8)
- removed the Echo1 at (128.3, 163.8)
- removed the Echo1 at (143.5, 127.0)
- removed the Echo1 at (48.3, 74.9)
- removed the Echo1 at (63.5, 38.1)
- removed the Echo1 at (222.2, 74.9)
- removed the Echo1 at (237.5, 38.1)
- removed the Echo1 at (146.1, 38.1)
- removed the Echo2 at (53.3, 161.3)
- removed the Echo2 at (135.9, 161.3)
- removed the Echo2 at (55.9, 72.4)
- removed the Echo2 at (229.9, 72.4)
- removed the Echo2 at (138.4, 72.4)
- removed the SalidasEcho1 at (69.8, 163.8)
- removed the SalidasEcho1 at (152.4, 163.8)
- removed the SalidasEcho1 at (72.4, 74.9)
- removed the SalidasEcho1 at (246.4, 74.9)
- removed the SalidasEcho1 at (154.9, 74.9)
- removed SalidasTrig1 (x5): Conn_01x08_Female, Connector_Molex:Molex_KK-254_AE-6410-08A_1x08_P2.54mm_Vertical
- removed Trig2 (x5): 74HCT137, Package_DIP:DIP-16_W7.62mm_LongPads
- added Echo1: Conn_01x01_Female, Connector_Molex:Molex_KK-254_AE-6410-06A_1x06_P2.54mm_Vertical, F.Cu at (232.4, 157.5)
- added Echo1: Conn_01x01_Female, Connector_Molex:Molex_KK-254_AE-6410-06A_1x06_P2.54mm_Vertical, F.Cu at (133.3, 157.5)
- added Echo1: Conn_01x01_Female, Connector_Molex:Molex_KK-254_AE-6410-06A_1x06_P2.54mm_Vertical, F.Cu at (40.6, 157.5)
- added Echo1: Conn_01x01_Female, Connector_Molex:Molex_KK-254_AE-6410-06A_1x06_P2.54mm_Vertical, F.Cu at (232.4, 63.5)
- added Echo1: Conn_01x01_Female, Connector_Molex:Molex_KK-254_AE-6410-06A_1x06_P2.54mm_Vertical, F.Cu at (133.3, 63.5)
- added Echo1: Conn_01x01_Female, Connector_Molex:Molex_KK-254_AE-6410-06A_1x06_P2.54mm_Vertical, F.Cu at (40.6, 63.5)
- added Echo2: 74LS151, Package_DIP:DIP-16_W7.62mm_LongPads, F.Cu at (149.9, 163.8)
- added Echo2: 74LS151, Package_DIP:DIP-16_W7.62mm_LongPads, F.Cu at (248.9, 163.8)
- added Echo2: 74LS151, Package_DIP:DIP-16_W7.62mm_LongPads, F.Cu at (57.1, 163.8)
- added Echo2: 74LS151, Package_DIP:DIP-16_W7.62mm_LongPads, F.Cu at (248.9, 69.8)
- added Echo2: 74LS151, Package_DIP:DIP-16_W7.62mm_LongPads, F.Cu at (149.9, 69.8)
- added Echo2: 74LS151, Package_DIP:DIP-16_W7.62mm_LongPads, F.Cu at (57.1, 69.8)
- added EntradasTrig1: Conn_01x08_Female, Connector_Molex:Molex_KK-254_AE-6410-08A_1x08_P2.54mm_Vertical, F.Cu at (259.1, 135.9)
- added EntradasTrig1: Conn_01x08_Female, Connector_Molex:Molex_KK-254_AE-6410-08A_1x08_P2.54mm_Vertical, F.Cu at (160.0, 135.9)
- added EntradasTrig1: Conn_01x08_Female, Connector_Molex:Molex_KK-254_AE-6410-08A_1x08_P2.54mm_Vertical, F.Cu at (67.3, 135.9)
- added EntradasTrig1: Conn_01x08_Female, Connector_Molex:Molex_KK-254_AE-6410-08A_1x08_P2.54mm_Vertical, F.Cu at (259.1, 41.9)
- added EntradasTrig1: Conn_01x08_Female, Connector_Molex:Molex_KK-254_AE-6410-08A_1x08_P2.54mm_Vertical, F.Cu at (160.0, 41.9)
- added EntradasTrig1: Conn_01x08_Female, Connector_Molex:Molex_KK-254_AE-6410-08A_1x08_P2.54mm_Vertical, F.Cu at (67.3, 41.9)
- added SalidasEcho1: Conn_01x08_Female, Connector_Molex:Molex_KK-254_AE-6410-08A_1x08_P2.54mm_Vertical, F.Cu at (160.0, 160.0)
- added SalidasEcho1: Conn_01x08_Female, Connector_Molex:Molex_KK-254_AE-6410-08A_1x08_P2.54mm_Vertical, F.Cu at (259.1, 160.0)
- added SalidasEcho1: Conn_01x08_Female, Connector_Molex:Molex_KK-254_AE-6410-08A_1x08_P2.54mm_Vertical, F.Cu at (67.3, 160.0)
- added SalidasEcho1: Conn_01x08_Female, Connector_Molex:Molex_KK-254_AE-6410-08A_1x08_P2.54mm_Vertical, F.Cu at (259.1, 66.0)
- added SalidasEcho1: Conn_01x08_Female, Connector_Molex:Molex_KK-254_AE-6410-08A_1x08_P2.54mm_Vertical, F.Cu at (160.0, 66.0)
- added SalidasEcho1: Conn_01x08_Female, Connector_Molex:Molex_KK-254_AE-6410-08A_1x08_P2.54mm_Vertical, F.Cu at (67.3, 66.0)
- added Trig1: Conn_01x01_Female, Connector_Molex:Molex_KK-254_AE-6410-02A_1x02_P2.54mm_Vertical, F.Cu at (248.9, 123.2)
- added Trig1: Conn_01x01_Female, Connector_Molex:Molex_KK-254_AE-6410-02A_1x02_P2.54mm_Vertical, F.Cu at (149.9, 123.2)
- added Trig1: Conn_01x01_Female, Connector_Molex:Molex_KK-254_AE-6410-02A_1x02_P2.54mm_Vertical, F.Cu at (57.1, 123.2)
- added Trig1: Conn_01x01_Female, Connector_Molex:Molex_KK-254_AE-6410-02A_1x02_P2.54mm_Vertical, F.Cu at (248.9, 29.2)
- added Trig1: Conn_01x01_Female, Connector_Molex:Molex_KK-254_AE-6410-02A_1x02_P2.54mm_Vertical, F.Cu at (149.9, 29.2)
- added Trig1: Conn_01x01_Female, Connector_Molex:Molex_KK-254_AE-6410-02A_1x02_P2.54mm_Vertical, F.Cu at (57.1, 29.2)
- added Trig3: 74HC237, Package_DIP:DIP-16_W7.62mm_LongPads, F.Cu at (146.1, 133.3)
- added Trig3: 74HC237, Package_DIP:DIP-16_W7.62mm_LongPads, F.Cu at (245.1, 133.3)
- added Trig3: 74HC237, Package_DIP:DIP-16_W7.62mm_LongPads, F.Cu at (53.3, 133.3)
- added Trig3: 74HC237, Package_DIP:DIP-16_W7.62mm_LongPads, F.Cu at (245.1, 39.4)
- added Trig3: 74HC237, Package_DIP:DIP-16_W7.62mm_LongPads, F.Cu at (146.1, 39.4)
- added Trig3: 74HC237, Package_DIP:DIP-16_W7.62mm_LongPads, F.Cu at (53.3, 39.4)
Routing:
- net Net-(Trig1-Pad1): track 49.9 -> 331.3 mm
- net Net-(Trig2-Pad1): track 0.00 -> 231.7 mm
- net Select1: track 188.9 -> 417.4 mm
- net Net-(Echo2-Pad4): track 0.00 -> 148.5 mm
- net 5V: track 317.0 -> 452.0 mm
- net Net-(Echo2-Pad3): track 0.00 -> 122.5 mm
- net Net-(Echo2-Pad12): track 44.4 -> 165.6 mm
- net Net-(EntradasTrig1-Pad8): track 0.00 -> 97.1 mm
- net Net-(SalidasTrig1-Pad8): track 96.9 -> 0.00 mm
- net Net-(Echo2-Pad2): track 0.00 -> 96.4 mm
- net Net-(Echo2-Pad13): track 44.4 -> 139.6 mm
- net Net-(Echo2-Pad7): track 93.1 -> 0.00 mm
- net Select2: track 277.7 -> 352.8 mm
- net Net-(Echo2-Pad14): track 44.4 -> 118.0 mm
- net Select3: track 347.2 -> 274.7 mm
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
Commit message: Actualizacion de placas
Parts:
- removed the Echo1 at (232.4, 157.5)
- removed the Echo1 at (133.3, 157.5)
- removed the Echo1 at (40.6, 157.5)
- removed the Echo1 at (232.4, 63.5)
- removed the Echo1 at (133.3, 63.5)
- removed the Echo2 at (149.9, 163.8)
- removed the Echo2 at (248.9, 163.8)
- removed the Echo2 at (57.1, 163.8)
- removed the Echo2 at (248.9, 69.8)
- removed the Echo2 at (149.9, 69.8)
- removed the EntradasTrig1 at (259.1, 135.9)
- removed the EntradasTrig1 at (160.0, 135.9)
- removed the EntradasTrig1 at (67.3, 135.9)
- removed the EntradasTrig1 at (259.1, 41.9)
- removed the EntradasTrig1 at (160.0, 41.9)
- removed the SalidasEcho1 at (160.0, 160.0)
- removed the SalidasEcho1 at (259.1, 160.0)
- removed the SalidasEcho1 at (67.3, 160.0)
- removed the SalidasEcho1 at (259.1, 66.0)
- removed the SalidasEcho1 at (160.0, 66.0)
- removed Trig1 (x6): Conn_01x01_Female, Connector_Molex:Molex_KK-254_AE-6410-02A_1x02_P2.54mm_Vertical
- removed the Trig3 at (146.1, 133.3)
- removed the Trig3 at (245.1, 133.3)
- removed the Trig3 at (53.3, 133.3)
- removed the Trig3 at (245.1, 39.4)
- removed the Trig3 at (146.1, 39.4)
- added 5V US: Conn_01x08_Female, Connector_Molex:Molex_KK-254_AE-6410-08A_1x08_P2.54mm_Vertical, F.Cu at (49.8, 93.0)
- added Alimentación: DOU, TerminalBlock:TerminalBlock_bornier-4_P5.08mm, F.Cu at (54.6, 32.5)
- added GND US: Conn_01x08_Female, Connector_Molex:Molex_KK-254_AE-6410-08A_1x08_P2.54mm_Vertical, F.Cu at (49.8, 85.9)
- added REF**: DOU, TerminalBlock:TerminalBlock_bornier-4_P5.08mm, F.Cu at (34.0, 32.5)
- moved EntradasTrig1 2.54 mm to (67.3, 44.5)
- moved Trig3 2.54 mm to (53.3, 41.9)
Routing:
- net Select1: track 417.4 -> 67.4 mm
- net Select2: track 352.8 -> 57.7 mm
- net 5V: track 452.0 -> 157.5 mm, vias 0 -> 2
- net Net-(Trig1-Pad1): track 331.3 -> 48.0 mm
- net Select3: track 274.7 -> 46.3 mm
- net Net-(Trig2-Pad1): track 231.7 -> 34.1 mm
- net Net-(Echo2-Pad12): track 165.6 -> 24.7 mm
- net Net-(Echo2-Pad4): track 148.5 -> 22.9 mm
- net Net-(Echo2-Pad13): track 139.6 -> 21.8 mm
- net Net-(Echo2-Pad3): track 122.5 -> 19.4 mm
- net Net-(Echo2-Pad14): track 118.0 -> 19.0 mm
- net Net-(EntradasTrig1-Pad8): track 97.1 -> 16.1 mm
- net Net-(Echo2-Pad2): track 96.4 -> 15.9 mm
- net Net-(Echo2-Pad15): track 96.4 -> 16.1 mm
- net Net-(Echo2-Pad1): track 70.4 -> 11.7 mm
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