File: Hardware/Circuito de Control de Marcha/Circuito de Control de Marcha.sch (KiCad schematic (older format))
At the start: 42 parts, among them Q1 IRF9540N, Q2 IRF540N, Q3 IRF9540N, Q4 IRF540N, Q5 IRF9540N, Q6 IRF540N, Q7 IRF9540N, Q8 IRF540N, U1 ULN2003, U2 4N25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

Commit message: CCM
agregue un mux en el puente del cangilon para controlarlo con un solo pwm
Parts:
- removed U2: 4N25, Package_DIP:DIP-6_W7.62mm, symbol Isolator:4N25
- added U10: 4N25, Package_DIP:DIP-6_W7.62mm, symbol Isolator:4N25
- added U2: 74LS157, Package_DIP:DIP-18_W7.62mm_LongPads, symbol 74xx:74LS157
- Bateria1: symbol Connector:Screw_Terminal_01x02 -> Connector:Screw_Terminal_01x03
Connections:
- net Earth: now also U10.2, U10.4, U2.15 (E), U2.2 (I0a), U2.6 (I1b), U2.8 (GND)
- net at R13.1, R2.2: now also U2.7 (Zb); no longer uC_Propulsion1.1 (Pin_1)
- net at R1.2, R14.1: now also U2.4 (Za); no longer uC_Propulsion1.2 (Pin_2)
- net at Q1.1 (G), R3.2: now also U10.5
- net at R1.1: now also U10.1
- new net: U2.1 (S), uC_Propulsion1.1 (Pin_1)
- new net: U2.3 (I1a), U2.5 (I0b), uC_Propulsion1.2 (Pin_2)
- new net 5V: Bateria1.3 (Pin_3), U2.16 (VCC)
Other:
- moved on the sheet: C1, F1, Motor_Cangilon1, Motor_Direccion1, Motor_Propulsion1, Q1, Q2, Q3, Q4, Q5, Q6, Q7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
