File: Hardware/Circuito de Control de Marcha/Circuito de Control de Marcha opto final.kicad_pcb (KiCad board)
At the start: 2 copper layers, 42 parts, among them Q1 IRF9540N, Q2 IRF540N, Q3 IRF9540N, Q4 IRF540N, Q5 IRF9540N, Q6 IRF540N, Q7 IRF9540N, Q8 IRF540N, U2 4N25, U3 4N25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

Commit message: CCM
agregue un mux en el puente del cangilon para controlarlo con un solo pwm
Parts:
- added U2: 74LS157, Package_DIP:DIP-18_W7.62mm_LongPads, F.Cu at (108.0, 83.8)
- Bateria1: footprint TerminalBlock:TerminalBlock_bornier-2_P5.08mm -> TerminalBlock:TerminalBlock_bornier-3_P5.08mm
- moved uC_Propulsion1 32.3 mm to (100.3, 92.7), turned to 270 degrees
- moved uCDireccion1 23.3 mm to (100.3, 115.6)
- moved uC_Cangilon1 12.0 mm to (100.3, 102.9)
- renumbered ULN2003 to U1
Connections:
- uC_Propulsion1 pad 1: Net-(R13-Pad1) -> Net-(U2-Pad1)
- uC_Propulsion1 pad 2: Net-(R1-Pad2) -> Net-(U2-Pad3)
Routing:
- net (no net): track 0.00 -> 43.5 mm
- net Net-(U2-Pad3): track 0.00 -> 32.1 mm
- net Net-(U1-Pad3): track 20.3 -> 48.4 mm
- net Net-(U1-Pad2): track 20.3 -> 48.4 mm
- net Net-(U1-Pad1): track 20.3 -> 48.4 mm
- net Net-(U1-Pad4): track 20.3 -> 47.6 mm
- net Net-(R1-Pad2): track 28.0 -> 51.5 mm
- net Net-(R16-Pad1): track 28.7 -> 41.9 mm
- net Net-(U2-Pad1): track 0.00 -> 12.8 mm
- net Net-(R15-Pad1): track 81.1 -> 92.8 mm
- net Net-(R13-Pad1): track 77.4 -> 80.0 mm

Commit message: Ultimos detalles CCM
Achique un poco la placa y la prepare para imprimir
Parts:
- moved C1 45.5 mm to (104.6, 137.2)
- moved U1 13.9 mm to (118.4, 126.0), turned to 270 degrees
- moved Motor_Direccion1 4.93 mm to (158.5, 133.1), turned to 90 degrees
- moved uCDireccion1 2.03 mm to (102.4, 115.6)
- moved uC_Cangilon1 2.03 mm to (102.4, 102.9)
- moved uC_Propulsion1 2.03 mm to (102.4, 92.7)
Routing:
- net Net-(Motor_Direccion1-Pad4): track 17.8 -> 61.1 mm
- net Net-(U1-Pad4): track 47.6 -> 13.9 mm
- net Net-(Motor_Direccion1-Pad3): track 17.8 -> 48.6 mm
- net Net-(C1-Pad1): track 357.2 -> 387.5 mm
- net Net-(U1-Pad3): track 48.4 -> 18.7 mm
- net Net-(Motor_Direccion1-Pad2): track 17.8 -> 45.0 mm
- net Net-(U1-Pad2): track 48.4 -> 22.3 mm
- net Net-(Motor_Direccion1-Pad1): track 17.8 -> 40.3 mm
- net Net-(U1-Pad1): track 48.4 -> 26.2 mm
- net Net-(R15-Pad1): track 92.8 -> 90.6 mm
- net Net-(R16-Pad1): track 41.9 -> 39.9 mm
- net Net-(U2-Pad3): track 32.1 -> 31.0 mm
- net Net-(U2-Pad1): track 12.8 -> 11.8 mm
